File: V1/esp-poe-2rl-V1-power.kicad_sch (KiCad schematic)
At the start: 32 parts, among them U4 TX4138, U5 SY8089A1AAC, U6 TPS2376DDAR-H

Commit message: addressing the PHY power rails
Parts:
- removed C22: 22uF/10V, Tales:C_1206_3216Metric, symbol Device:C_Small
- C18: value 10uF/10V -> 10uF/25V; footprint Tales:C_0603_1608Metric -> Tales:C_0805_2012Metric; LCSC Part # C19702 -> C15850; Mfr PN CL10A106KP8NNNC -> CL21A106KAYNNNE; Package 0603/1608 -> 0805/2012; Vendor PN C19702 -> C15850
- R28: LCSC Part # C60490 -> C25744; Mfr Yageo -> Uniroyal
Other:
- moved on the sheet: C25

Commit message: Replaced terminal blocks
Parts:
- R34: renamed from R28; Mfr PN RC0402FR-0710KL -> 0402WGF1002TCE; Vendor PN C60490 -> C25744
- renumbered C17 to C21, C23 to C22, C19 to C23, C21 to C24, C24 to C25, C20 to C26, C25 to C27, C18 to C28, D9 to D10, D10 to D11, D11 to D8, D8 to D9, R22 to R31, R27 to R32, R21 to R33, R31 to R35, R23 to R36, R24 to R37, R19 to R38, R29 to R39, R30 to R40, R25 to R41, R20 to R42, R26 to R43, U6 to U4, U4 to U5, U5 to U6

Commit message: V1.5.0
Parts:
- L2: footprint Tales:L_12x12mm_h6mm -> Tales:L_12x12mm_H6mm
- L3: footprint Tales:L_3x3mm_h1.5mm -> Tales:L_3x3mm_H1.5mm
Changed lines of the file:
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@@
 			)
 		)
-		(property "Footprint" "Tales:L_3x3mm_h1.5mm"
+		(property "Footprint" "Tales:L_3x3mm_H1.5mm"
 			(at 102.87 148.59 0)
 			(hide yes)
@@
 			)
 		)
-		(property "Footprint" "Tales:L_12x12mm_h6mm"
+		(property "Footprint" "Tales:L_12x12mm_H6mm"
 			(at 101.6 96.52 0)
 			(hide yes)

Commit message: Revising before manufacture
Changed lines of the file:
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@@
 	(wire
 		(pts
-			(xy 48.26 106.68) (xy 48.26 93.98)
+			(xy 48.26 107.95) (xy 48.26 93.98)
 		)
 		(stroke
@@
 	(wire
 		(pts
-			(xy 43.18 106.68) (xy 48.26 106.68)
+			(xy 24.13 107.95) (xy 48.26 107.95)
 		)
 		(stroke
@@
 	(global_label "PG"
 		(shape input)
-		(at 43.18 106.68 180)
+		(at 24.13 107.95 180)
 		(fields_autoplaced yes)
 		(effects
@@
 		)
 		(property "Intersheetrefs" "${INTERSHEET_REFS}"
-			(at 37.7342 106.68 0)
+			(at 18.6842 107.95 0)
 			(hide yes)
 			(show_name no)
@@
 			(at 44.45 185.42 0)
 			(hide yes)
+			(show_name no)
+			(do_not_autoplace no)
+			(effects
+				(font
+					(size 1.27 1.27)
+				)
+			)
+		)
+		(property "Sim.Pins" "1=K 2=A"
+			(at 44.45 185.42 0)
+			(hide yes)
