File: V1/esp-poe-2rl-V1.kicad_pcb (KiCad board)
At the start: 4 copper layers, 82.5 x 45 mm, 105 parts, among them J1 USB_C_Receptacle_USB2.0, J2 250-202, J3 RJ45 JACK, J4 250-202, K1 G5NB-1A-E-DC5, K2 G5NB-1A-E-DC5, Q1 UMH3N, Q2 MMBT2222A, Q3 WPM2015-3/TR, Q4 LMUN2211LT1G, Q5 MMBT2222A, SW1 RESET, U1 CH340K, U2 ESP32-WROOM-32UE-N16, U3 LAN8710A, U4 TPS2376DDAR-H, U5 TX4138, U6 SY8089A1AAC

Commit message: Update resistance value for pull-ups.
Parts:
- R2: value 10k -> 1.5k
- R3, R4, R5, R6, R7, R8, R9: value 10k -> 2.2k
Changed lines of the file:
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@@
 			)
 		)
-		(property "Value" "10k"
+		(property "Value" "2.2k"
 			(at 0 1.17 0)
 			(layer "F.Fab")
@@
 			)
 		)
-		(property "Mfr PN" "0402WGF1002TCE"
+		(property "Mfr PN" "0402WGF2201TCE"
 			(at 0 0 180)
 			(unlocked yes)
@@
 			)
 		)
-		(property "Vendor PN" "C25744"
+		(property "Vendor PN" "C25879"
 			(at 0 0 180)
 			(unlocked yes)
@@
 			)
 		)
-		(property "LCSC Part #" "C25744"
+		(property "LCSC Part #" "C25879"
 			(at 0 0 180)
 			(unlocked yes)
@@
 			(unit
 				(name "A")
-				(pins "3" "4" "5" "21" "22" "17" "18" "20" "19" "32" "2" "1" "38" "39"
-					"15" "25" "35" "24" "34" "26" "29" "14" "16" "13" "23" "27" "28" "30"
+				(pins "3" "4" "5" "21" "22" "17" "18" "20" "19" "32" "2" "1" "38" "15"
+					"39" "25" "35" "24" "34" "26" "29" "14" "16" "13" "23" "27" "28" "30"
 					"31" "33" "36" "37" "10" "11" "12" "8" "9" "6" "7"
 				)
@@
 			)
 		)
-		(property "Value" "10k"
+		(property "Value" "2.2k"
 			(at 0 1.17 90)
 			(layer "F.Fab")
@@
 			)
 		)
-		(property "Mfr PN" "0402WGF1002TCE"
+		(property "Mfr PN" "0402WGF2201TCE"
 			(at 0 0 270)
 			(unlocked yes)
@@
 			)
 		)
-		(property "Vendor PN" "C25744"
+		(property "Vendor PN" "C25879"
 			(at 0 0 270)
 			(unlocked yes)
@@
 			)
 		)
-		(property "LCSC Part #" "C25744"
+		(property "LCSC Part #" "C25879"
 			(at 0 0 270)
 			(unlocked yes)
@@
 			)
 		)
-		(property "Value" "10k"
+		(property "Value" "2.2k"
 			(at 0 1.17 90)
 			(layer "F.Fab")
@@
 			)
 		)
-		(property "Mfr PN" "0402WGF1002TCE"
+		(property "Mfr PN" "0402WGF2201TCE"
 			(at 0 0 270)
 			(unlocked yes)
@@
 			)
 		)
-		(property "Vendor PN" "C25744"
+		(property "Vendor PN" "C25879"
 			(at 0 0 270)
 			(unlocked yes)
@@
 			)
 		)
-		(property "LCSC Part #" "C25744"
+		(property "LCSC Part #" "C25879"
 			(at 0 0 270)
 			(unlocked yes)
@@
 			)
 		)
-		(property "Value" "10k"
+		(property "Value" "1.5k"
 			(at 0 1.17 90)
 			(layer "F.Fab")
@@
 			)
 		)
-		(property "Mfr PN" "0402WGF1002TCE"
+		(property "Mfr PN" "0402WGF1501TCE"
 			(at 0 0 270)
 			(unlocked yes)
@@
 			)
 		)
-		(property "Vendor PN" "C25744"
+		(property "Vendor PN" "C25867"
 			(at 0 0 270)
 			(unlocked yes)
@@
 			)
 		)
-		(property "LCSC Part #" "C25744"
+		(property "LCSC Part #" "C25867"
 			(at 0 0 270)
 			(unlocked yes)
@@
 			)
 		)
-		(property "Value" "10k"
+		(property "Value" "2.2k"
 			(at 0 1.17 90)
 			(layer "F.Fab")
@@
 			)
 		)
-		(property "Mfr PN" "0402WGF1002TCE"
+		(property "Mfr PN" "0402WGF2201TCE"
 			(at 0 0 270)
 			(unlocked yes)
@@
 			)
 		)
-		(property "Vendor PN" "C25744"
+		(property "Vendor PN" "C25879"
 			(at 0 0 270)
 			(unlocked yes)
@@
 			)
 		)
-		(property "LCSC Part #" "C25744"
+		(property "LCSC Part #" "C25879"
 			(at 0 0 270)
 			(unlocked yes)
@@
 			)
 		)
-		(property "Value" "10k"
+		(property "Value" "2.2k"
 			(at 0 1.17 90)
 			(layer "F.Fab")
@@
 			)
 		)
-		(property "Mfr PN" "0402WGF1002TCE"
+		(property "Mfr PN" "0402WGF2201TCE"
 			(at 0 0 270)
 			(unlocked yes)
@@
 			)
 		)
-		(property "Vendor PN" "C25744"
+		(property "Vendor PN" "C25879"
 			(at 0 0 270)
 			(unlocked yes)
@@
 			)
 		)
-		(property "LCSC Part #" "C25744"
+		(property "LCSC Part #" "C25879"
 			(at 0 0 270)
 			(unlocked yes)
@@
 			)
 		)
-		(property "Value" "10k"
+		(property "Value" "2.2k"
 			(at 0 1.17 90)
 			(layer "F.Fab")
@@
 			)
 		)
-		(property "Mfr PN" "0402WGF1002TCE"
+		(property "Mfr PN" "0402WGF2201TCE"
 			(at 0 0 270)
 			(unlocked yes)
@@
 			)
 		)
-		(property "Vendor PN" "C25744"
+		(property "Vendor PN" "C25879"
 			(at 0 0 270)
 			(unlocked yes)
@@
 			)
 		)
-		(property "LCSC Part #" "C25744"
+		(property "LCSC Part #" "C25879"
 			(at 0 0 270)
 			(unlocked yes)
@@
 			)
 		)
-		(property "Value" "10k"
+		(property "Value" "2.2k"
 			(at 0 1.17 0)
 			(layer "F.Fab")
@@
 			)
 		)
-		(property "Mfr PN" "0402WGF1002TCE"
+		(property "Mfr PN" "0402WGF2201TCE"
 			(at 0 0 180)
 			(unlocked yes)
@@
 			)
 		)
-		(property "Vendor PN" "C25744"
+		(property "Vendor PN" "C25879"
 			(at 0 0 180)
 			(unlocked yes)
@@
 			)
 		)
-		(property "LCSC Part #" "C25744"
+		(property "LCSC Part #" "C25879"
 			(at 0 0 180)
 			(unlocked yes)
@@
 		(target_length 33.4)
 		(target_length_max 33.5)
-		(target_length_min 33.3)
+		(target_length_min 33.299999)
 		(target_skew 0)
 		(target_skew_max 0.1)
@@
 		(last_status "tuned")
 		(last_track_width 0.2)
-		(last_tuning_length 33.396159)
+		(last_tuning_length 33.396158)
 		(max_amplitude 0.85)
 		(min_amplitude 0.2)

Commit message: Revising before manufacture
Connections:
- net /OUT1BJT renamed /RELAY OUTPUTS/OUT1BJT
- net /OUT1CMD renamed /RELAY OUTPUTS/OUT1CMD
- net /OUT1LD renamed /RELAY OUTPUTS/OUT1LD
- net /OUT1LN renamed /RELAY OUTPUTS/OUT1LN
- net /OUT1ON renamed /RELAY OUTPUTS/OUT1ON
- net /OUT2BJT renamed /RELAY OUTPUTS/OUT2BJT
- net /OUT2CMD renamed /RELAY OUTPUTS/OUT2CMD
- net /OUT2LD renamed /RELAY OUTPUTS/OUT2LD
- net /OUT2LN renamed /RELAY OUTPUTS/OUT2LN
- net /OUT2ON renamed /RELAY OUTPUTS/OUT2ON

Commit message: V1.4.0
Other:
- board text added: "ESP-POE-2RL V1"
- board text added: "V1.4.0 2026-06-10"
- board text removed: "ESP-POE-2RL V1.5"
- board text removed: "V1.5.0 2026-06-08"
