File: V1/esp-poe-2rl-V1.kicad_pcb (KiCad board)
At the start: 4 copper layers, 82.5 x 45 mm, 105 parts, among them J1 USB_C_Receptacle_USB2.0, J2 250-202, J3 RJ45 JACK, J4 250-202, K1 G5NB-1A-E-DC5, K2 G5NB-1A-E-DC5, Q1 UMH3N, Q2 MMBT2222A, Q3 WPM2015-3/TR, Q4 LMUN2211LT1G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

Commit message: Streamlining version numbers.
Other:
- board text added: "V1.4 2026-06-10"
- board text removed: "V1.4.0 2026-06-10"
Changed lines of the file:
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@@
 	(gr_rect
 		(start 135.75 113.5)
-		(end 147.25 115.25)
+		(end 146.25 115.25)
 		(stroke
 			(width 0.1)
@@
 		)
 	)
-	(gr_text "V1.4.0 2026-06-10"
-		(at 136 115 0)
+	(gr_text "V1.4 2026-06-10"
+		(at 141 114.375 0)
 		(layer "F.SilkS")
 		(effects
@@
 				(thickness 0.1)
 			)
-			(justify left bottom)
 		)
 	)
