File: V1/eumesmo-poe-2rl-v1-outputs.kicad_sch (KiCad schematic)
At the start: 16 parts, among them J2 250-202, J4 250-202, K1 G5NB-1A-E-DC5, K2 G5NB-1A-E-DC5, Q2 MMBT2222A, Q5 MMBT2222A

Commit message: Renamed all files to eumesmo branding
Other:
- title: (none) -> eumesmo 2x Relay Output Module with PoE
Changed lines of the file:
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@@
 	(paper "A4")
 	(title_block
-		(rev "V1.4")
+		(title "eumesmo 2x Relay Output Module with PoE")
+		(date "2026-06-13")
+		(rev "V1.5")
 	)
 	(junction
@@
 		)
 		(instances
-			(project "esp-poe-2rl-V1"
+			(project "eumesmo-poe-2rl-V1"
 				(path "/2bc5a21a-1d79-419d-a592-6852cc07b00a/774cc362-9cfe-4197-8571-7d1b1ef33e48"
 					(reference "R21")
@@
 		)
 		(instances
-			(project "esp-poe-2rl-V1"
+			(project "eumesmo-poe-2rl-V1"
 				(path "/2bc5a21a-1d79-419d-a592-6852cc07b00a/774cc362-9cfe-4197-8571-7d1b1ef33e48"
 					(reference "K2")
@@
 		)
 		(instances
-			(project "esp-poe-2rl-V1"
+			(project "eumesmo-poe-2rl-V1"
 				(path "/2bc5a21a-1d79-419d-a592-6852cc07b00a/774cc362-9cfe-4197-8571-7d1b1ef33e48"
 					(reference "D4")
@@
 		)
 		(instances
-			(project "esp-poe-2rl-V1"
+			(project "eumesmo-poe-2rl-V1"
 				(path "/2bc5a21a-1d79-419d-a592-6852cc07b00a/774cc362-9cfe-4197-8571-7d1b1ef33e48"
 					(reference "D5")
@@
 		)
 		(instances
-			(project "esp-poe-2rl-V1"
+			(project "eumesmo-poe-2rl-V1"
 				(path "/2bc5a21a-1d79-419d-a592-6852cc07b00a/774cc362-9cfe-4197-8571-7d1b1ef33e48"
 					(reference "D3")
@@
 		)
 		(instances
-			(project "esp-poe-2rl-V1"
+			(project "eumesmo-poe-2rl-V1"
 				(path "/2bc5a21a-1d79-419d-a592-6852cc07b00a/774cc362-9cfe-4197-8571-7d1b1ef33e48"
 					(reference "#PWR055")
@@
 		)
 		(instances
-			(project "esp-poe-2rl-V1"
+			(project "eumesmo-poe-2rl-V1"
 				(path "/2bc5a21a-1d79-419d-a592-6852cc07b00a/774cc362-9cfe-4197-8571-7d1b1ef33e48"
 					(reference "R23")
@@
 		)
 		(instances
-			(project "esp-poe-2rl-V1"
+			(project "eumesmo-poe-2rl-V1"
 				(path "/2bc5a21a-1d79-419d-a592-6852cc07b00a/774cc362-9cfe-4197-8571-7d1b1ef33e48"
 					(reference "R27")
@@
 		)
 		(instances
-			(project "esp-poe-2rl-V1"
+			(project "eumesmo-poe-2rl-V1"
 				(path "/2bc5a21a-1d79-419d-a592-6852cc07b00a/774cc362-9cfe-4197-8571-7d1b1ef33e48"
 					(reference "#PWR039")
@@
 		)
 		(instances
-			(project "esp-poe-2rl-V1"
+			(project "eumesmo-poe-2rl-V1"
 				(path "/2bc5a21a-1d79-419d-a592-6852cc07b00a/774cc362-9cfe-4197-8571-7d1b1ef33e48"
 					(reference "J2")
@@
 		)
 		(instances
-			(project "esp-poe-2rl-V1"
+			(project "eumesmo-poe-2rl-V1"
 				(path "/2bc5a21a-1d79-419d-a592-6852cc07b00a/774cc362-9cfe-4197-8571-7d1b1ef33e48"
 					(reference "R30")
@@
 		)
 		(instances
-			(project "esp-poe-2rl-V1"
+			(project "eumesmo-poe-2rl-V1"
 				(path "/2bc5a21a-1d79-419d-a592-6852cc07b00a/774cc362-9cfe-4197-8571-7d1b1ef33e48"
 					(reference "Q5")
@@
 		)
 		(instances
-			(project "esp-poe-2rl-V1"
+			(project "eumesmo-poe-2rl-V1"
 				(path "/2bc5a21a-1d79-419d-a592-6852cc07b00a/774cc362-9cfe-4197-8571-7d1b1ef33e48"
 					(reference "#PWR047")
@@
 		)
 		(instances
-			(project "esp-poe-2rl-V1"
+			(project "eumesmo-poe-2rl-V1"
 				(path "/2bc5a21a-1d79-419d-a592-6852cc07b00a/774cc362-9cfe-4197-8571-7d1b1ef33e48"
 					(reference "#PWR046")
@@
 		)
 		(instances
-			(project "esp-poe-2rl-V1"
+			(project "eumesmo-poe-2rl-V1"
 				(path "/2bc5a21a-1d79-419d-a592-6852cc07b00a/774cc362-9cfe-4197-8571-7d1b1ef33e48"
 					(reference "J4")
@@
 		)
 		(instances
-			(project "esp-poe-2rl-V1"
+			(project "eumesmo-poe-2rl-V1"
 				(path "/2bc5a21a-1d79-419d-a592-6852cc07b00a/774cc362-9cfe-4197-8571-7d1b1ef33e48"
 					(reference "R22")
@@
 		)
 		(instances
-			(project "esp-poe-2rl-V1"
+			(project "eumesmo-poe-2rl-V1"
 				(path "/2bc5a21a-1d79-419d-a592-6852cc07b00a/774cc362-9cfe-4197-8571-7d1b1ef33e48"
 					(reference "#PWR044")
@@
 		)
 		(instances
-			(project "esp-poe-2rl-V1"
+			(project "eumesmo-poe-2rl-V1"
 				(path "/2bc5a21a-1d79-419d-a592-6852cc07b00a/774cc362-9cfe-4197-8571-7d1b1ef33e48"
 					(reference "K1")
@@
 		)
 		(instances
-			(project "esp-poe-2rl-V1"
+			(project "eumesmo-poe-2rl-V1"
 				(path "/2bc5a21a-1d79-419d-a592-6852cc07b00a/774cc362-9cfe-4197-8571-7d1b1ef33e48"
 					(reference "#PWR054")
@@
 		)
 		(instances
-			(project "esp-poe-2rl-V1"
+			(project "eumesmo-poe-2rl-V1"
 				(path "/2bc5a21a-1d79-419d-a592-6852cc07b00a/774cc362-9cfe-4197-8571-7d1b1ef33e48"
 					(reference "Q2")
@@
 		)
 		(instances
-			(project "esp-poe-2rl-V1"
+			(project "eumesmo-poe-2rl-V1"
 				(path "/2bc5a21a-1d79-419d-a592-6852cc07b00a/774cc362-9cfe-4197-8571-7d1b1ef33e48"
 					(reference "R29")
@@
 		)
 		(instances
-			(project "esp-poe-2rl-V1"
+			(project "eumesmo-poe-2rl-V1"
 				(path "/2bc5a21a-1d79-419d-a592-6852cc07b00a/774cc362-9cfe-4197-8571-7d1b1ef33e48"
 					(reference "D6")
