File: V1/eumesmo-poe-2rl-v1-outputs.kicad_sch (KiCad schematic)
At the start: 16 parts, among them J2 250-202, J4 250-202, K1 G5NB-1A-E-DC5, K2 G5NB-1A-E-DC5, Q2 MMBT2222A, Q5 MMBT2222A

Commit message: Added CPU health LED
Parts:
- renumbered D4 to D10, D5 to D11, D6 to D12, D3 to D9, J2 to J3, Q2 to Q4, R21 to R39, R22 to R40, R23 to R41, R27 to R42, R29 to R43, R30 to R44
Connections:
- net OUT1LD: now also J3.1 (Pin_1); no longer J3.2 (Pin_2)
- net OUT1LN: now also J3.2 (Pin_2); no longer J3.1 (Pin_1)
- net OUT2LD: now also J4.1 (Pin_1); no longer J4.2 (Pin_2)
- net OUT2LN: now also J4.2 (Pin_2); no longer J4.1 (Pin_1)
Other:
- moved on the sheet: J3, J4
