File: V1/eumesmo-poe-2rl-v1-power.kicad_sch (KiCad schematic)
At the start: 31 parts, among them U4 TPS2376DDAR-H, U5 TX4138, U6 SY8089A1AAC

Commit message: Renamed all files to eumesmo branding
Other:
- title: ESP 2x Relay Output Module with PoE -> eumesmo 2x Relay Output Module with PoE
Changed lines of the file:
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@@
 	(paper "A4")
 	(title_block
-		(title "ESP 2x Relay Output Module with PoE")
-		(date "2026-01-29")
-		(rev "V1.4")
+		(title "eumesmo 2x Relay Output Module with PoE")
+		(date "2026-06-13")
+		(rev "V1.5")
 	)
 	(text "R_{TPS1}"
@@
 		)
 		(instances
-			(project "esp-poe-2rl-V1"
+			(project "eumesmo-poe-2rl-V1"
 				(path "/2bc5a21a-1d79-419d-a592-6852cc07b00a/2ac7b96d-5459-407c-a3e3-5692241632df"
 					(reference "#PWR069")
@@
 		)
 		(instances
-			(project "esp-poe-2rl-V1"
+			(project "eumesmo-poe-2rl-V1"
 				(path "/2bc5a21a-1d79-419d-a592-6852cc07b00a/2ac7b96d-5459-407c-a3e3-5692241632df"
 					(reference "R37")
@@
 		)
 		(instances
-			(project "esp-poe-2rl-V1"
+			(project "eumesmo-poe-2rl-V1"
 				(path "/2bc5a21a-1d79-419d-a592-6852cc07b00a/2ac7b96d-5459-407c-a3e3-5692241632df"
 					(reference "#PWR056")
@@
 		)
 		(instances
-			(project "esp-poe-2rl-V1"
+			(project "eumesmo-poe-2rl-V1"
 				(path "/2bc5a21a-1d79-419d-a592-6852cc07b00a/2ac7b96d-5459-407c-a3e3-5692241632df"
 					(reference "C23")
@@
 		)
 		(instances
-			(project "esp-poe-2rl-V1"
+			(project "eumesmo-poe-2rl-V1"
 				(path "/2bc5a21a-1d79-419d-a592-6852cc07b00a/2ac7b96d-5459-407c-a3e3-5692241632df"
 					(reference "R40")
@@
 		)
 		(instances
-			(project "esp-poe-2rl-V1"
+			(project "eumesmo-poe-2rl-V1"
 				(path "/2bc5a21a-1d79-419d-a592-6852cc07b00a/2ac7b96d-5459-407c-a3e3-5692241632df"
 					(reference "#PWR063")
@@
 		)
 		(instances
-			(project "esp-poe-2rl-V1"
+			(project "eumesmo-poe-2rl-V1"
 				(path "/2bc5a21a-1d79-419d-a592-6852cc07b00a/2ac7b96d-5459-407c-a3e3-5692241632df"
 					(reference "L3")
@@
 		)
 		(instances
-			(project "esp-poe-2rl-V1"
+			(project "eumesmo-poe-2rl-V1"
 				(path "/2bc5a21a-1d79-419d-a592-6852cc07b00a/2ac7b96d-5459-407c-a3e3-5692241632df"
 					(reference "C21")
@@
 		)
 		(instances
-			(project "esp-poe-2rl-V1"
+			(project "eumesmo-poe-2rl-V1"
 				(path "/2bc5a21a-1d79-419d-a592-6852cc07b00a/2ac7b96d-5459-407c-a3e3-5692241632df"
 					(reference "C27")
@@
 		)
 		(instances
-			(project "esp-poe-2rl-V1"
+			(project "eumesmo-poe-2rl-V1"
 				(path "/2bc5a21a-1d79-419d-a592-6852cc07b00a/2ac7b96d-5459-407c-a3e3-5692241632df"
 					(reference "#PWR061")
@@
 		)
 		(instances
-			(project "esp-poe-2rl-V1"
+			(project "eumesmo-poe-2rl-V1"
 				(path "/2bc5a21a-1d79-419d-a592-6852cc07b00a/2ac7b96d-5459-407c-a3e3-5692241632df"
 					(reference "#PWR066")
@@
 		)
 		(instances
-			(project "esp-poe-2rl-V1"
+			(project "eumesmo-poe-2rl-V1"
 				(path "/2bc5a21a-1d79-419d-a592-6852cc07b00a/2ac7b96d-5459-407c-a3e3-5692241632df"
 					(reference "D9")
@@
 		)
 		(instances
-			(project "esp-poe-2rl-V1"
+			(project "eumesmo-poe-2rl-V1"
 				(path "/2bc5a21a-1d79-419d-a592-6852cc07b00a/2ac7b96d-5459-407c-a3e3-5692241632df"
 					(reference "R32")
@@
 		)
 		(instances
-			(project "esp-poe-2rl-V1"
+			(project "eumesmo-poe-2rl-V1"
 				(path "/2bc5a21a-1d79-419d-a592-6852cc07b00a/2ac7b96d-5459-407c-a3e3-5692241632df"
 					(reference "L2")
@@
 		)
 		(instances
-			(project "esp-poe-2rl-V1"
+			(project "eumesmo-poe-2rl-V1"
 				(path "/2bc5a21a-1d79-419d-a592-6852cc07b00a/2ac7b96d-5459-407c-a3e3-5692241632df"
 					(reference "R35")
@@
 		)
 		(instances
-			(project "esp-poe-2rl-V1"
+			(project "eumesmo-poe-2rl-V1"
 				(path "/2bc5a21a-1d79-419d-a592-6852cc07b00a/2ac7b96d-5459-407c-a3e3-5692241632df"
 					(reference "C26")
@@
 		)
 		(instances
-			(project "esp-poe-2rl-V1"
+			(project "eumesmo-poe-2rl-V1"
 				(path "/2bc5a21a-1d79-419d-a592-6852cc07b00a/2ac7b96d-5459-407c-a3e3-5692241632df"
 					(reference "U4")
@@
 		)
 		(instances
-			(project "esp-poe-2rl-V1"
+			(project "eumesmo-poe-2rl-V1"
 				(path "/2bc5a21a-1d79-419d-a592-6852cc07b00a/2ac7b96d-5459-407c-a3e3-5692241632df"
 					(reference "C22")
@@
 		)
 		(instances
-			(project "esp-poe-2rl-V1"
+			(project "eumesmo-poe-2rl-V1"
 				(path "/2bc5a21a-1d79-419d-a592-6852cc07b00a/2ac7b96d-5459-407c-a3e3-5692241632df"
 					(reference "#FLG05")
@@
 		)
 		(instances
-			(project "esp-poe-2rl-V1"
+			(project "eumesmo-poe-2rl-V1"
 				(path "/2bc5a21a-1d79-419d-a592-6852cc07b00a/2ac7b96d-5459-407c-a3e3-5692241632df"
 					(reference "R33")
@@
 		)
 		(instances
-			(project "esp-poe-2rl-V1"
+			(project "eumesmo-poe-2rl-V1"
 				(path "/2bc5a21a-1d79-419d-a592-6852cc07b00a/2ac7b96d-5459-407c-a3e3-5692241632df"
 					(reference "#PWR059")
@@
 		)
 		(instances
-			(project "esp-poe-2rl-V1"
+			(project "eumesmo-poe-2rl-V1"
 				(path "/2bc5a21a-1d79-419d-a592-6852cc07b00a/2ac7b96d-5459-407c-a3e3-5692241632df"
 					(reference "D8")
@@
 		)
 		(instances
-			(project "esp-poe-2rl-V1"
+			(project "eumesmo-poe-2rl-V1"
 				(path "/2bc5a21a-1d79-419d-a592-6852cc07b00a/2ac7b96d-5459-407c-a3e3-5692241632df"
 					(reference "#PWR065")
@@
 		)
 		(instances
-			(project "esp-poe-2rl-V1"
+			(project "eumesmo-poe-2rl-V1"
 				(path "/2bc5a21a-1d79-419d-a592-6852cc07b00a/2ac7b96d-5459-407c-a3e3-5692241632df"
 					(reference "R31")
@@
 		)
 		(instances
-			(project "esp-poe-2rl-V1"
+			(project "eumesmo-poe-2rl-V1"
 				(path "/2bc5a21a-1d79-419d-a592-6852cc07b00a/2ac7b96d-5459-407c-a3e3-5692241632df"
 					(reference "#PWR058")
@@
 		)
 		(instances
-			(project "esp-poe-2rl-V1"
+			(project "eumesmo-poe-2rl-V1"
 				(path "/2bc5a21a-1d79-419d-a592-6852cc07b00a/2ac7b96d-5459-407c-a3e3-5692241632df"
 					(reference "R39")
@@
 		)
 		(instances
-			(project "esp-poe-2rl-V1"
+			(project "eumesmo-poe-2rl-V1"
 				(path "/2bc5a21a-1d79-419d-a592-6852cc07b00a/2ac7b96d-5459-407c-a3e3-5692241632df"
 					(reference "R41")
@@
 		)
 		(instances
-			(project "esp-poe-2rl-V1"
+			(project "eumesmo-poe-2rl-V1"
 				(path "/2bc5a21a-1d79-419d-a592-6852cc07b00a/2ac7b96d-5459-407c-a3e3-5692241632df"
 					(reference "R36")
@@
 		)
 		(instances
-			(project "esp-poe-2rl-V1"
+			(project "eumesmo-poe-2rl-V1"
 				(path "/2bc5a21a-1d79-419d-a592-6852cc07b00a/2ac7b96d-5459-407c-a3e3-5692241632df"
 					(reference "R38")
@@
 		)
 		(instances
-			(project "esp-poe-2rl-V1"
+			(project "eumesmo-poe-2rl-V1"
 				(path "/2bc5a21a-1d79-419d-a592-6852cc07b00a/2ac7b96d-5459-407c-a3e3-5692241632df"
 					(reference "R34")
@@
 		)
 		(instances
-			(project "esp-poe-2rl-V1"
+			(project "eumesmo-poe-2rl-V1"
 				(path "/2bc5a21a-1d79-419d-a592-6852cc07b00a/2ac7b96d-5459-407c-a3e3-5692241632df"
 					(reference "D7")
@@
 		)
 		(instances
-			(project "esp-poe-2rl-V1"
+			(project "eumesmo-poe-2rl-V1"
 				(path "/2bc5a21a-1d79-419d-a592-6852cc07b00a/2ac7b96d-5459-407c-a3e3-5692241632df"
 					(reference "D11")
@@
 		)
 		(instances
-			(project "esp-poe-2rl-V1"
+			(project "eumesmo-poe-2rl-V1"
 				(path "/2bc5a21a-1d79-419d-a592-6852cc07b00a/2ac7b96d-5459-407c-a3e3-5692241632df"
 					(reference "R42")
@@
 		)
 		(instances
-			(project "esp-poe-2rl-V1"
+			(project "eumesmo-poe-2rl-V1"
 				(path "/2bc5a21a-1d79-419d-a592-6852cc07b00a/2ac7b96d-5459-407c-a3e3-5692241632df"
 					(reference "U5")
@@
 		)
 		(instances
-			(project "esp-poe-2rl-V1"
+			(project "eumesmo-poe-2rl-V1"
 				(path "/2bc5a21a-1d79-419d-a592-6852cc07b00a/2ac7b96d-5459-407c-a3e3-5692241632df"
 					(reference "#PWR062")
@@
 		)
 		(instances
-			(project "esp-poe-2rl-V1"
+			(project "eumesmo-poe-2rl-V1"
 				(path "/2bc5a21a-1d79-419d-a592-6852cc07b00a/2ac7b96d-5459-407c-a3e3-5692241632df"
 					(reference "R43")
@@
 		)
 		(instances
-			(project "esp-poe-2rl-V1"
+			(project "eumesmo-poe-2rl-V1"
 				(path "/2bc5a21a-1d79-419d-a592-6852cc07b00a/2ac7b96d-5459-407c-a3e3-5692241632df"
 					(reference "#PWR060")
@@
 		)
 		(instances
-			(project "esp-poe-2rl-V1"
+			(project "eumesmo-poe-2rl-V1"
 				(path "/2bc5a21a-1d79-419d-a592-6852cc07b00a/2ac7b96d-5459-407c-a3e3-5692241632df"
 					(reference "#PWR068")
@@
 		)
 		(instances
-			(project "esp-poe-2rl-V1"
+			(project "eumesmo-poe-2rl-V1"
 				(path "/2bc5a21a-1d79-419d-a592-6852cc07b00a/2ac7b96d-5459-407c-a3e3-5692241632df"
 					(reference "C24")
@@
 		)
 		(instances
-			(project "esp-poe-2rl-V1"
+			(project "eumesmo-poe-2rl-V1"
 				(path "/2bc5a21a-1d79-419d-a592-6852cc07b00a/2ac7b96d-5459-407c-a3e3-5692241632df"
 					(reference "U6")
@@
 		)
 		(instances
-			(project "esp-poe-2rl-V1"
+			(project "eumesmo-poe-2rl-V1"
 				(path "/2bc5a21a-1d79-419d-a592-6852cc07b00a/2ac7b96d-5459-407c-a3e3-5692241632df"
 					(reference "#PWR067")
@@
 		)
 		(instances
-			(project "esp-poe-2rl-V1"
+			(project "eumesmo-poe-2rl-V1"
 				(path "/2bc5a21a-1d79-419d-a592-6852cc07b00a/2ac7b96d-5459-407c-a3e3-5692241632df"
 					(reference "C25")
@@
 		)
 		(instances
-			(project "esp-poe-2rl-V1"
+			(project "eumesmo-poe-2rl-V1"
 				(path "/2bc5a21a-1d79-419d-a592-6852cc07b00a/2ac7b96d-5459-407c-a3e3-5692241632df"
 					(reference "D10")
@@
 		)
 		(instances
-			(project "esp-poe-2rl-V1"
+			(project "eumesmo-poe-2rl-V1"
 				(path "/2bc5a21a-1d79-419d-a592-6852cc07b00a/2ac7b96d-5459-407c-a3e3-5692241632df"
 					(reference "#PWR057")
@@
 		)
 		(instances
-			(project "esp-poe-2rl-V1"
+			(project "eumesmo-poe-2rl-V1"
 				(path "/2bc5a21a-1d79-419d-a592-6852cc07b00a/2ac7b96d-5459-407c-a3e3-5692241632df"
 					(reference "C28")
@@
 		)
 		(instances
-			(project "esp-poe-2rl-V1"
+			(project "eumesmo-poe-2rl-V1"
 				(path "/2bc5a21a-1d79-419d-a592-6852cc07b00a/2ac7b96d-5459-407c-a3e3-5692241632df"
 					(reference "#PWR064")
@@
 		)
 		(instances
-			(project "esp-poe-2rl-V1"
+			(project "eumesmo-poe-2rl-V1"
 				(path "/2bc5a21a-1d79-419d-a592-6852cc07b00a/2ac7b96d-5459-407c-a3e3-5692241632df"
 					(reference "#FLG04")
