File: V1/eumesmo-poe-2rl-v1.kicad_sch (KiCad schematic)
At the start: 56 parts, among them J1 USB_C_Receptacle_USB2.0, J3 RJ45 JACK, Q1 UMH3N, Q3 WPM2015-3/TR, Q4 LMUN2211LT1G, SW1 RESET, U1 CH340K, U2 ESP32-WROOM-32UE-N16, U3 LAN8710A

Commit message: Renamed all files to eumesmo branding
Other:
- sheet POWER: file esp-poe-2rl-v1-power.kicad_sch -> eumesmo-poe-2rl-V1-power.kicad_sch
- sheet RELAY OUTPUTS: file esp-poe-2rl-v1-outputs.kicad_sch -> eumesmo-poe-2rl-V1-outputs.kicad_sch
- note added: "ESP32 TEMPLATE FOR GPIO ASSIGNMENT {"NAME":"eumesmo-poe-2rl-v1","GPIO":[0,3200,0,3232,0,0,0,0,5536,224,0,0,225,0,5600,0,0,0,0,5568,0,0,0,0,0,0,0,0,608,640,0,0,0,0,0,0],"FLAG":0,"BASE":1} https://tasmota.github.io/docs/Templates/"
- note removed: "ESP32 TEMPLATE FOR GPIO ASSIGNMENT {"NAME":"ESP-POE-2RL-V1","GPIO":[0,3200,0,3232,0,0,0,0,5536,224,0,0,225,0,5600,0,0,0,0,5568,0,0,0,0,0,0,0,0,608,640,0,0,0,0,0,0],"FLAG":0,"BASE":1} https://tasmota.github.io/docs/Templates/"
- title: ESP 2x Relay Output Module with PoE -> eumesmo 2x Relay Output Module with PoE
